File: monitoreo_solar/monitoreo_solar.kicad_sch (KiCad schematic)
At the start: 25 parts, among them J1 Screw_Terminal_01x02, J2 Conn_01x03_Socket, J3 Screw_Terminal_01x02, J4 Conn_01x04_Pin, J5 Conn_01x03_Pin, U1 X9C103S, U2 AMS1117-3.3, U4 LM358

Commit message: first pcb design
Parts:
- H1, H2, H3, H4: footprint MountingHole:MountingHole_5mm -> MountingHole:MountingHole_3.2mm_M3
Connections:
- net Vout is gone; now on net Pot+: R3.1
- net +3.3V: now also J4.1 (Pin_1); no longer J4.4 (Pin_4)
- net DIR: now also J5.3 (Pin_3); no longer J5.2 (Pin_2)
- net GND: now also J4.4 (Pin_4); no longer J4.1 (Pin_1)
- net STEP: now also J5.2 (Pin_2); no longer J5.3 (Pin_3)
Changed lines of the file:
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@@
 	(wire
 		(pts
-			(xy 29.21 25.4) (xy 35.56 25.4)
+			(xy 151.13 69.85) (xy 143.51 69.85)
 		)
 		(stroke
@@
 	(wire
 		(pts
-			(xy 143.51 77.47) (xy 143.51 81.28)
+			(xy 29.21 25.4) (xy 35.56 25.4)
 		)
 		(stroke
@@
 	(wire
 		(pts
+			(xy 143.51 69.85) (xy 143.51 81.28)
+		)
+		(stroke
+			(width 0)
+			(type default)
+		)
+	)
+	(wire
+		(pts
 			(xy 73.66 39.37) (xy 73.66 41.91)
 		)
@@
 	(wire
 		(pts
-			(xy 143.51 88.9) (xy 143.51 92.71)
+			(xy 143.51 88.9) (xy 143.51 99.06)
 		)
 		(stroke
@@
 	(wire
 		(pts
-			(xy 109.22 33.02) (xy 109.22 36.83)
+			(xy 143.51 99.06) (xy 151.13 99.06)
 		)
 		(stroke
@@
 	(wire
 		(pts
-			(xy 100.33 167.64) (xy 106.68 167.64)
+			(xy 109.22 33.02) (xy 109.22 36.83)
 		)
 		(stroke
@@
 	(wire
 		(pts
+			(xy 151.13 73.66) (xy 151.13 69.85)
+		)
+		(stroke
+			(width 0)
+			(type default)
+		)
+	)
+	(wire
+		(pts
 			(xy 52.07 72.39) (xy 52.07 63.5)
 		)
@@
 	(wire
 		(pts
+			(xy 100.33 167.64) (xy 106.68 167.64)
+		)
+		(stroke
+			(width 0)
+			(type default)
+		)
+	)
+	(wire
+		(pts
+			(xy 100.33 163.83) (xy 104.14 163.83)
+		)
+		(stroke
+			(width 0)
+			(type default)
+		)
+	)
+	(wire
+		(pts
 			(xy 104.14 163.83) (xy 104.14 165.1)
 		)
@@
 	(wire
 		(pts
+			(xy 151.13 99.06) (xy 151.13 96.52)
+		)
+		(stroke
+			(width 0)
+			(type default)
+		)
+	)
+	(wire
+		(pts
 			(xy 29.21 49.53) (xy 35.56 49.53)
 		)
@@
 		)
 	)
-	(wire
-		(pts
-			(xy 100.33 163.83) (xy 104.14 163.83)
-		)
-		(stroke
-			(width 0)
-			(type default)
-		)
-	)
 	(global_label "Vcurrent"
 		(shape input)
@@
 	(global_label "STEP"
 		(shape input)
-		(at 100.33 163.83 180)
+		(at 100.33 167.64 180)
 		(fields_autoplaced yes)
 		(effects
@@
 		)
 		(property "Intersheetrefs" "${INTERSHEET_REFS}"
-			(at 92.7487 163.83 0)
+			(at 92.7487 167.64 0)
 			(effects
 				(font
@@
 		)
 	)
-	(global_label "Vout"
+	(global_label "Vamp2"
 		(shape input)
 		(at 93.98 97.79 180)
@@
 		)
 		(property "Intersheetrefs" "${INTERSHEET_REFS}"
-			(at 86.8825 97.79 0)
+			(at 84.7054 97.79 0)
 			(effects
 				(font
@@
 	(global_label "DIR"
 		(shape input)
-		(at 100.33 167.64 180)
+		(at 100.33 163.83 180)
 		(fields_autoplaced yes)
 		(effects
@@
 		)
 		(property "Intersheetrefs" "${INTERSHEET_REFS}"
-			(at 94.2 167.64 0)
+			(at 94.2 163.83 0)
 			(effects
 				(font
@@
 			)
 		)
-		(property "Footprint" "MountingHole:MountingHole_5mm"
+		(property "Footprint" "MountingHole:MountingHole_3.2mm_M3"
 			(at 199.39 27.94 0)
 			(effects
@@
 	(symbol
 		(lib_id "power:+3.3V")
-		(at 143.51 77.47 0)
+		(at 113.03 46.99 0)
 		(unit 1)
 		(exclude_from_sim no)
@@
 		(dnp no)
 		(fields_autoplaced yes)
-		(property "Reference" "#PWR06"
-			(at 143.51 81.28 0)
+		(property "Reference" "#PWR04"
+			(at 113.03 50.8 0)
 			(effects
 				(font
@@
 		)
 		(property "Value" "+3.3V"
-			(at 143.51 72.39 0)
+			(at 113.03 41.91 0)
 			(effects
 				(font
@@
 		)
 		(property "Footprint" ""
-			(at 143.51 77.47 0)
+			(at 113.03 46.99 0)
 			(effects
 				(font
@@
 		)
 		(property "Datasheet" ""
-			(at 143.51 77.47 0)
+			(at 113.03 46.99 0)
 			(effects
 				(font
@@
 		)
 		(property "Description" "Power symbol creates a global label with name \"+3.3V\""
-			(at 143.51 77.47 0)
+			(at 113.03 46.99 0)
 			(effects
 				(font
@@
 			(project "monitoreo_solar"
 				(path "/51bfdde5-5428-4bd6-badc-0ec3b16e1032"
-					(reference "#PWR06")
+					(reference "#PWR04")
 					(unit 1)
 				)
@@
 	)
 	(symbol
-		(lib_id "power:+3.3V")
-		(at 113.03 46.99 0)
+		(lib_id "power:GND")
+		(at 151.13 73.66 0)
 		(unit 1)
 		(exclude_from_sim no)
@@
 		(dnp no)
 		(fields_autoplaced yes)
-		(property "Reference" "#PWR04"
-			(at 113.03 50.8 0)
+		(property "Reference" "#PWR07"
+			(at 151.13 80.01 0)
 			(effects
 				(font
@@
 			)
 		)
-		(property "Value" "+3.3V"
-			(at 113.03 41.91 0)
+		(property "Value" "GND"
+			(at 151.13 78.74 0)
 			(effects
 				(font
@@
 		)
 		(property "Footprint" ""
-			(at 113.03 46.99 0)
+			(at 151.13 73.66 0)
 			(effects
 				(font
@@
 		)
 		(property "Datasheet" ""
-			(at 113.03 46.99 0)
+			(at 151.13 73.66 0)
 			(effects
 				(font
@@
 			)
 		)
-		(property "Description" "Power symbol creates a global label with name \"+3.3V\""
-			(at 113.03 46.99 0)
+		(property "Description" "Power symbol creates a global label with name \"GND\" , ground"
+			(at 151.13 73.66 0)
 			(effects
 				(font
@@
 			(project "monitoreo_solar"
 				(path "/51bfdde5-5428-4bd6-badc-0ec3b16e1032"
-					(reference "#PWR04")
+					(reference "#PWR07")
 					(unit 1)
 				)
@@
 			)
 		)
-		(property "Footprint" "MountingHole:MountingHole_5mm"
+		(property "Footprint" "MountingHole:MountingHole_3.2mm_M3"
 			(at 199.39 38.1 0)
 			(effects
@@
 	)
 	(symbol
-		(lib_id "power:GND")
-		(at 143.51 92.71 0)
-		(unit 1)
-		(exclude_from_sim no)
-		(in_bom yes)
-		(on_board yes)
-		(dnp no)
-		(fields_autoplaced yes)
-		(property "Reference" "#PWR07"
-			(at 143.51 99.06 0)
-			(effects
-				(font
-					(size 1.27 1.27)
-				)
-				(hide yes)
-			)
-		)
-		(property "Value" "GND"
-			(at 143.51 97.79 0)
-			(effects
-				(font
-					(size 1.27 1.27)
-				)
-			)
-		)
-		(property "Footprint" ""
-			(at 143.51 92.71 0)
-			(effects
-				(font
-					(size 1.27 1.27)
-				)
-				(hide yes)
-			)
-		)
-		(property "Datasheet" ""
-			(at 143.51 92.71 0)
-			(effects
-				(font
-					(size 1.27 1.27)
-				)
-				(hide yes)
-			)
-		)
-		(property "Description" "Power symbol creates a global label with name \"GND\" , ground"
-			(at 143.51 92.71 0)
-			(effects
-				(font
-					(size 1.27 1.27)
-				)
-				(hide yes)
-			)
-		)
-		(pin "1"
-		)
-		(instances
-			(project "monitoreo_solar"
-				(path "/51bfdde5-5428-4bd6-badc-0ec3b16e1032"
-					(reference "#PWR07")
-					(unit 1)
-				)
-			)
-		)
-	)
-	(symbol
 		(lib_id "Mechanical:MountingHole")
 		(at 199.39 22.86 0)
@@
 			)
 		)
-		(property "Footprint" "MountingHole:MountingHole_5mm"
+		(property "Footprint" "MountingHole:MountingHole_3.2mm_M3"
 			(at 199.39 22.86 0)
 			(effects
@@
 	)
 	(symbol
+		(lib_id "power:+3.3V")
+		(at 151.13 96.52 0)
+		(unit 1)
+		(exclude_from_sim no)
+		(in_bom yes)
+		(on_board yes)
+		(dnp no)
+		(property "Reference" "#PWR06"
+			(at 151.13 100.33 0)
+			(effects
+				(font
+					(size 1.27 1.27)
+				)
+				(hide yes)
+			)
+		)
+		(property "Value" "+3.3V"
+			(at 151.13 91.44 0)
+			(effects
+				(font
+					(size 1.27 1.27)
+				)
+			)
+		)
+		(property "Footprint" ""
+			(at 151.13 96.52 0)
+			(effects
+				(font
+					(size 1.27 1.27)
+				)
+				(hide yes)
+			)
+		)
+		(property "Datasheet" ""
+			(at 151.13 96.52 0)
+			(effects
+				(font
+					(size 1.27 1.27)
+				)
+				(hide yes)
+			)
+		)
+		(property "Description" "Power symbol creates a global label with name \"+3.3V\""
+			(at 151.13 96.52 0)
+			(effects
+				(font
+					(size 1.27 1.27)
+				)
+				(hide yes)
+			)
+		)
+		(pin "1"
+		)
+		(instances
+			(project "monitoreo_solar"
+				(path "/51bfdde5-5428-4bd6-badc-0ec3b16e1032"
+					(reference "#PWR06")
+					(unit 1)
+				)
+			)
+		)
+	)
+	(symbol
 		(lib_id "power:GND")
 		(at 54.61 137.16 0)
@@
 			)
 		)
-		(property "Footprint" "MountingHole:MountingHole_5mm"
+		(property "Footprint" "MountingHole:MountingHole_3.2mm_M3"
 			(at 199.39 33.02 0)
 			(effects
@@
 		(on_board yes)
 		(dnp no)
-		(fields_autoplaced yes)
 		(property "Reference" "J1"
 			(at 24.13 43.18 0)
